Commit message: added lane keeping CV algorithm

File: src/description_2602_foxtrot/ackermann_urdf/camera.xacro (robot description, xacro)
@@ -24,5 +24,5 @@
         <child link="camera_link"/>
         <!-- Placed at the front of the chassis. Adjust X and Z as necessary -->
-        <origin xyz="0.1 0 0.1" rpy="0 0 0"/>
+        <origin xyz="0.0 0 0.0" rpy="0 0 0"/>
     </joint>
     <!-- Virtual Optical Link for ROS 2 Image Data Convention -->

File: src/description_2602_foxtrot/diffdrive_urdf/camera.xacro (robot description, xacro)
@@ -43,5 +43,6 @@
             <gz_frame_id>camera_link_optical</gz_frame_id>
             <camera>
-                <horizontal_fov>1.089</horizontal_fov> <!-- Approx 62 degrees -->
+                <!-- Widened to 1.57 radians (90 degrees) for peripheral vision -->
+                <horizontal_fov>1.57</horizontal_fov>
                 <image>
                     <width>640</width>
@@ -51,5 +52,5 @@
                 <clip>
                     <near>0.05</near>
-                    <far>8.0</far>
+                    <far>15.0</far> <!-- Extended view distance -->
                 </clip>
                 <noise>
